Commit message: Velocity control working without PID implementation

File: src/description/arm.urdf (robot description, URDF)
Before this commit: robot None, 4 links, 3 joints
Links:
- added link world
Joints:
- added joint world_fixed: type fixed, parent world, child base_link, origin xyz=0.0 0.0 0.0 rpy=0.0 0.0 0.0, axis 0.0 0.0 0.0, limit lower=0.0 upper=0.0 effort=0.0 velocity=0.0

File: src/description/arm_sim.ros2_control.xacro (robot description, xacro)
@@ -4,8 +4,8 @@
     <ros2_control name = "ArmSystem" type="system">
         <hardware>
-            <plugin>mock_components/GenericSystem</plugin>
+            <plugin>gazebo_ros2_control/GazeboSystem</plugin>
         </hardware>
         <joint name="base_joint">
-            <command_interface name="position"></command_interface>
+            <command_interface name="velocity"></command_interface>
             <state_interface name="position"></state_interface>
             <state_interface name="velocity"></state_interface>
@@ -13,5 +13,5 @@
         </joint>
         <joint name="first_arm_joint">
-            <command_interface name="position"></command_interface>
+            <command_interface name="velocity"></command_interface>
             <state_interface name="position"></state_interface>
             <state_interface name="velocity"></state_interface>
@@ -19,5 +19,5 @@
         </joint>
         <joint name="second_arm_joint">
-            <command_interface name="position"></command_interface>
+            <command_interface name="velocity"></command_interface>
             <state_interface name="position"></state_interface>
             <state_interface name="velocity"></state_interface>

Commit message: Revert "Velocity control working without PID implementation"
This reverts commit 281510653e25e1a3b63ff957f5f906f9e1864a26.

File: src/description/arm.urdf (robot description, URDF)
Before this commit: robot None, 5 links, 4 joints
Links:
- removed link world
Joints:
- removed joint world_fixed

File: src/description/arm_sim.ros2_control.xacro (robot description, xacro)
@@ -4,8 +4,8 @@
     <ros2_control name = "ArmSystem" type="system">
         <hardware>
-            <plugin>gazebo_ros2_control/GazeboSystem</plugin>
+            <plugin>mock_components/GenericSystem</plugin>
         </hardware>
         <joint name="base_joint">
-            <command_interface name="velocity"></command_interface>
+            <command_interface name="position"></command_interface>
             <state_interface name="position"></state_interface>
             <state_interface name="velocity"></state_interface>
@@ -13,5 +13,5 @@
         </joint>
         <joint name="first_arm_joint">
-            <command_interface name="velocity"></command_interface>
+            <command_interface name="position"></command_interface>
             <state_interface name="position"></state_interface>
             <state_interface name="velocity"></state_interface>
@@ -19,5 +19,5 @@
         </joint>
         <joint name="second_arm_joint">
-            <command_interface name="velocity"></command_interface>
+            <command_interface name="position"></command_interface>
             <state_interface name="position"></state_interface>
             <state_interface name="velocity"></state_interface>

Commit message: Position node running with gazebo_ros2_control simulation

File: src/description/arm.urdf (robot description, URDF)
Before this commit: robot None, 4 links, 3 joints
Links:
- added link world
Joints:
- added joint world_to_base: type fixed, parent world, child base_link, origin xyz=0.0 0.0 0.0 rpy=0.0 0.0 0.0
- joint first_arm_joint: axis (none) -> 0.0 1.0 0.0

File: src/description/arm_sim.ros2_control.xacro (robot description, xacro)
@@ -4,8 +4,11 @@
     <ros2_control name = "ArmSystem" type="system">
         <hardware>
-            <plugin>mock_components/GenericSystem</plugin>
+            <plugin>gazebo_ros2_control/GazeboSystem</plugin>
         </hardware>
         <joint name="base_joint">
-            <command_interface name="position"></command_interface>
+            <command_interface name="position">
+                <param name="min">-3.14</param>
+                <param name="max">3.14</param>
+            </command_interface>
             <state_interface name="position"></state_interface>
             <state_interface name="velocity"></state_interface>
@@ -13,5 +16,8 @@
         </joint>
         <joint name="first_arm_joint">
-            <command_interface name="position"></command_interface>
+            <command_interface name="position">
+                <param name="min">-0.7</param>
+                <param name="max">0.7</param>
+            </command_interface>
             <state_interface name="position"></state_interface>
             <state_interface name="velocity"></state_interface>
@@ -19,5 +25,8 @@
         </joint>
         <joint name="second_arm_joint">
-            <command_interface name="position"></command_interface>
+            <command_interface name="position">
+                <param name="min">-0.7</param>
+                <param name="max">0.7</param>
+            </command_interface>
             <state_interface name="position"></state_interface>
             <state_interface name="velocity"></state_interface>
@@ -29,5 +38,5 @@
       <plugin filename="libgazebo_ros2_control.so" name="gazebo_ros2_control">
         <!-- Path to ros params file for ros2_controllers-->
-        <parameters>Arm_Sim/src/config/my_controllers.yaml</parameters>
+        <parameters>/home/rushhaank/arm_sim/install/armsim/share/armsim/config/my_controllers.yaml</parameters>
       </plugin>
     </gazebo>
